File: microdrill/schematics/drill.sch (KiCad schematic (older format))
At the start: 12 parts, among them P1 CONN_2, P2 CONN_2, P3 CONN_2, Q1 MOS_N, U1 LM555N

Commit message: Added alpha-version of schematic + beginning of code (drill)
Parts:
- removed C1: 1u, symbol C
- removed P2, P3: CONN_2, symbol CONN_2
- removed Q1: MOS_N, symbol MOS_N
- removed R2: 1k, ~, symbol R
- removed RV1: POT, symbol POT
- removed U1: LM555N, symbol LM555N
- added R?: 1R, symbol R
- added VT?: S8205A, TSSOP-8, symbol S8205A
- R4: renamed from R1; value 10k -> 1k
- gave numbers to parts that had none: 1
- renumbered P1 to P7, R3 to R5, R4 to R6
Connections:
- net GND: now also R?.2
- net at R5.1, R6.1: now also R4.2, R?.1, VT?.2 (S1), VT?.3 (S1), VT?.5 (S2), VT?.7 (S2)
- net at D3.1 (A), P7.2 (PM): now also VT?.1 (D), VT?.8 (D)
- net VCC renamed Sence
- new net PWM_in: VT?.4 (G1), VT?.5 (S2)
Other:
- moved on the sheet: D3, P7, R4, R5, R6
