File: microdrill/schematics/MCU_module.sch (KiCad schematic (older format))
At the start: 29 parts, among them K1 POWER, P1 CONN_14, P2 CONN_4, P3 Stepper, P4 Slide, P5 CONN_14, P6 CONN_5, SW1 DRILL, SW2 BTN1, SW3 BTN2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

Commit message: added PCB for microdrill
Parts:
- removed C1: 1u, symbol C
- removed C2, C3: 104, symbol C
- removed D1, D2: LED, symbol LED
- removed P1, P5: CONN_14, symbol CONN_14
- removed P2: CONN_4, symbol CONN_4
- removed P6: CONN_5, symbol CONN_5
- removed R1, R2: 1k, symbol R
- removed R3: 10k, symbol R
- removed RV1: POT, symbol POT
- removed SW1: DRILL, ~, symbol SW_PUSH
- removed SW2: BTN1, ~, symbol SW_PUSH
- removed SW3: BTN2, ~, symbol SW_PUSH
- removed SW4: SW_PUSH, symbol SW_PUSH
- removed SW5: UP, ~, symbol SW_PUSH
- removed SW6: DOWN, ~, symbol SW_PUSH
- removed U1: STM8S105K4T6C, ~, symbol STM8S105K4T6C
- added BTN1, BTN2, DOWN1, DRILL+1, DRILL-1, DRILLSW1, GND1, POT1, UP1: CONN_1, symbol CONN_1
- added X1: STM8S105BOARD, devboard_pins-9-14, symbol STM8S105BOARD
Connections:
- net labels removed: 3.3V, 5.0V, RXD, TXD
- wire segments 100 -> 69
- no-connect marks 1 -> 12
Other:
- note added: ""DRILLSW" is foot-switch.\nPress it to move drill down,\nrelease to return it to start position.\nDouble-click turns drill motor on/off.\n"
- note added: "Drill motor + pedal"
- note added: "Tray"
- note removed: ""DRILL" is foot-switch.\nPress it to move drill down,\nrelease to return it to start position.\nDouble-click turns drill motor on/off.\n"
- note removed: "Drill motor"
- note removed: "STM8 board"
- note removed: "Slider (tray) motor"
- note removed: "USB <-> TTL"

Commit message: started voltmeter hacking
Parts:
- removed X1: STM8S105BOARD, devboard_pins-9-14, symbol STM8S105BOARD
- added X1: stm8s105board, devboard_pins-9-14, symbol stm8s105board
Changed lines of the file:
@@
 LIBS:s8205a
 LIBS:MCU_module-cache
-EELAYER 27 0
+EELAYER 24 0
 EELAYER END
 $Descr A3 16535 11693
@@
 Wire Notes Line
 	5300 2000 5300 1850
-$Comp
-L STM8S105BOARD X1
-U 1 1 54626F55
-P 3550 2350
-F 0 "X1" H 3550 3400 60  0000 C CNN
-F 1 "STM8S105BOARD" H 3550 1700 60  0000 C CNN
-F 2 "devboard_pins-9-14" H 3550 2350 60  0001 C CNN
-F 3 "~" H 3550 2350 60  0000 C CNN
-	1    3550 2350
-	1    0    0    -1
-$EndComp
 Wire Wire Line
 	1600 1650 1600 1600
@@
 Wire Wire Line
 	5450 6000 5750 6000
+$Comp
+L stm8s105board X1
+U 1 1 549FF443
+P 3550 2350
+F 0 "X1" H 3550 3400 60  0000 C CNN
+F 1 "stm8s105board" H 3550 1700 60  0000 C CNN
+F 2 "devboard_pins-9-14" H 3550 2350 60  0001 C CNN
+F 3 "" H 3550 2350 60  0000 C CNN
+	1    3550 2350
+	1    0    0    -1
+$EndComp
 $EndSCHEMATC
